Commit message: working in rviz2 and gazebo

File: scout_description/urdf/scout_v2/scout_v2.urdf (robot description, URDF)
Before this commit: robot scout_v2, 7 links, 6 joints
Joints:
- joint front_left_wheel: limit (none) -> effort=0.1 velocity=10.0
- joint front_right_wheel: limit (none) -> effort=0.1 velocity=10.0
- joint rear_left_wheel: limit (none) -> effort=0.1 velocity=10.0
- joint rear_right_wheel: limit (none) -> effort=0.1 velocity=10.0

File: scout_description/urdf/scout_v2/scout_v2.xacro (robot description, xacro)
@@ -62,8 +62,8 @@
     </xacro:scout_wheel_type1>
     <xacro:scout_wheel_type2 wheel_prefix="front_left">
-        <origin xyz="${wheelbase/2} ${track/2} ${wheel_vertical_offset}" rpy="0 0 0" />
+        <origin xyz="${wheelbase/2} ${track/2} ${wheel_vertical_offset}" rpy="3.14 0 0" />
     </xacro:scout_wheel_type2>
     <xacro:scout_wheel_type1 wheel_prefix="rear_left">
-        <origin xyz="${-wheelbase/2} ${track/2} ${wheel_vertical_offset}" rpy="0 0 0" />
+        <origin xyz="${-wheelbase/2} ${track/2} ${wheel_vertical_offset}" rpy="3.14 0 0" />
     </xacro:scout_wheel_type1>
     <xacro:scout_wheel_type2 wheel_prefix="rear_right">
